File: hardware/iot/iot.kicad_pcb (KiCad board)
At the start: 2 copper layers, 21 parts, among them J1 Conn_02x04_Top_Bottom, J2 Conn_01x02, J3 Conn_01x03, J4 Conn_01x03, SW1 SW_Push_SPDT, U1 WS2812b, U2 WS2812b, U3 WS2812b, U4 WS2812b, U5 WS2812b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

Commit message: Últimos cambios
Parts:
- added G***: LOGO, iot:logo, F.Cu at (140.5, 129.3)
- added REF**: MountingHole_3.2mm_M3, Mounting_Holes:MountingHole_3.2mm_M3, F.Cu at (122.4, 127.5)
- added REF**: MountingHole_3.2mm_M3, Mounting_Holes:MountingHole_3.2mm_M3, F.Cu at (156.7, 127.5)
- moved C2 68.7 mm to (135.6, 121.4)
- moved C8 68.2 mm to (135.6, 108.0)
- moved U6 67.9 mm to (125.0, 102.9), turned to 180 degrees
- moved C4 60.9 mm to (127.0, 114.3), turned to 90 degrees
- moved RX 60.0 mm to (121.9, 120.4), turned to 90 degrees
- moved C3 57.3 mm to (135.4, 116.8)
- moved U5 56.4 mm to (145.3, 125.5)
- moved R1 55.6 mm to (143.0, 114.6), turned to 90 degrees
- moved C6 52.9 mm to (140.0, 114.6), turned to 90 degrees
- moved C5 52.4 mm to (135.4, 112.0)
- moved TX 49.3 mm to (121.9, 108.2), turned to 90 degrees
- moved DHT11 48.2 mm to (157.2, 110.2)
- moved C7 45.1 mm to (145.3, 108.0)
- moved U1 43.3 mm to (135.6, 103.6), turned to 0 degrees
- moved J1 43.1 mm to (148.9, 111.0)
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- renumbered U7 to DHT11, J3 to RX, J4 to TX
Routing:
- net GND: track 0.00 -> 122.4 mm, vias 0 -> 1
- net +5V: track 0.00 -> 106.4 mm, vias 0 -> 3
- net +3V3: track 0.00 -> 51.2 mm, vias 0 -> 1
- net /TX: track 0.00 -> 44.6 mm
- net /RX: track 0.00 -> 34.3 mm, vias 0 -> 4
- net Net-(U2-Pad2): track 0.00 -> 28.3 mm, vias 0 -> 2
- net /GPIO_2: track 0.00 -> 22.3 mm, vias 0 -> 2
- net Net-(U4-Pad2): track 0.00 -> 21.6 mm, vias 0 -> 2
- net Net-(U3-Pad2): track 0.00 -> 21.4 mm, vias 0 -> 2
- net Net-(U1-Pad2): track 0.00 -> 17.0 mm, vias 0 -> 2
- net /CH_PD: track 0.00 -> 16.2 mm, vias 0 -> 2
- net /GPIO_0: track 0.00 -> 15.2 mm
- added copper zone on B.Cu, net GND
- added copper zone on F.Cu, net GND
Other:
- board outline added: 40.4 x 32.3 mm
- board text added: "+"
- board text added: "-"
- board text added: "OFF"
- board text added: "ON"
