File: hardware/iot/iot.sch (KiCad schematic (older format))
At the start: 21 parts, among them J1 Conn_02x04_Top_Bottom, J2 Conn_01x02, J3 Conn_01x03, J4 Conn_01x03, SW1 SW_Push_SPDT, U1 WS2812b, U2 WS2812b, U3 WS2812b, U4 WS2812b, U5 WS2812b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

Commit message: Últimos cambios
Changed lines of the file:
@@
 Wire Wire Line
 	6100 7000 6100 7250
+Wire Wire Line
+	5700 7000 5700 7250
 $EndSCHEMATC
